Commit message: Temp: hardware interface

File: ros/ros2_ws/src/doteacher/description/ros2_control/ros2_control_ackermann_drive.xacro (robot description, xacro)
@@ -1,5 +1,43 @@
 <?xml version="1.0"?>
 <robot xmlns:xacro="http://ros.org/wiki/xacro">
-    <ros2_control name="GazeboSystem" type="system">
+    <ros2_control name="RealRobot" type="system">
+        <hardware>
+            <plugin>doteacher/AckermannJetsonHardware</plugin>
+            <param name="rear_left_wheel">rear_left_wheel_joint</param>
+            <param name="rear_right_wheel">rear_right_wheel_joint</param>
+            <param name="front_left_wheel">front_left_steer_joint</param>
+            <param name="front_right_wheel">front_right_steer_joint</param>
+            <param name="loop_rate">20</param>
+        </hardware>
+        <joint name="rear_left_wheel_joint">
+            <command_interface name="velocity">
+                <param name="min">-1</param>
+                <param name="max">1</param>
+            </command_interface>
+            <state_interface name="velocity"/>
+        </joint>
+        <joint name="rear_right_wheel_joint">
+            <command_interface name="velocity">
+                <param name="min">-1</param>
+                <param name="max">1</param>
+            </command_interface>
+            <state_interface name="velocity"/>
+        </joint>
+        <joint name="front_left_steer_joint">
+            <command_interface name="position">
+                <param name="min">-0.5236</param>
+                <param name="max">0.5236</param>
+            </command_interface>
+            <state_interface name="position"/>
+        </joint>
+        <joint name="front_right_steer_joint">
+            <command_interface name="position">
+                <param name="min">-0.5236</param>
+                <param name="max">0.5236</param>
+            </command_interface>
+            <state_interface name="position"/>
+        </joint>
+    </ros2_control>
+    <!-- <ros2_control name="GazeboSystem" type="system">
         <hardware>
             <plugin>gazebo_ros2_control/GazeboSystem</plugin>
@@ -33,5 +71,5 @@
             <state_interface name="position"/>
         </joint>
-    </ros2_control>
+    </ros2_control> -->
     <gazebo>
         <plugin name="gazebo_ros2_control" filename="libgazebo_ros2_control.so">

File: ros/ros2_ws/src/doteacher/description/urdf/doteacher.urdf.xacro (robot description, xacro)
@@ -3,4 +3,6 @@
 <robot xmlns:xacro="http://www.ros.org/wiki/xacro" name="doteacher_robot">
   <xacro:arg name="prefix" default="" />
+  <xacro:arg name="use_ros2_control" default="true"/>
+  <xacro:arg name="sim_mode" default="false"/>
   <xacro:include filename="$(find doteacher)/urdf/doteacher_description.urdf.xacro" />
   <!-- Import Rviz colors -->

Commit message: Chore: launch 및 params 파일 추가

File: ros/ros2_ws/src/doteacher/description/ros2_control/ros2_control_ackermann_drive.xacro (robot description, xacro)
@@ -1,78 +1,83 @@
 <?xml version="1.0"?>
 <robot xmlns:xacro="http://ros.org/wiki/xacro">
-    <ros2_control name="RealRobot" type="system">
-        <hardware>
-            <plugin>doteacher/AckermannJetsonHardware</plugin>
-            <param name="rear_left_wheel">rear_left_wheel_joint</param>
-            <param name="rear_right_wheel">rear_right_wheel_joint</param>
-            <param name="front_left_wheel">front_left_steer_joint</param>
-            <param name="front_right_wheel">front_right_steer_joint</param>
-            <param name="loop_rate">20</param>
-        </hardware>
-        <joint name="rear_left_wheel_joint">
-            <command_interface name="velocity">
-                <param name="min">-1</param>
-                <param name="max">1</param>
-            </command_interface>
-            <state_interface name="velocity"/>
-        </joint>
-        <joint name="rear_right_wheel_joint">
-            <command_interface name="velocity">
-                <param name="min">-1</param>
-                <param name="max">1</param>
-            </command_interface>
-            <state_interface name="velocity"/>
-        </joint>
-        <joint name="front_left_steer_joint">
-            <command_interface name="position">
-                <param name="min">-0.5236</param>
-                <param name="max">0.5236</param>
-            </command_interface>
-            <state_interface name="position"/>
-        </joint>
-        <joint name="front_right_steer_joint">
-            <command_interface name="position">
-                <param name="min">-0.5236</param>
-                <param name="max">0.5236</param>
-            </command_interface>
-            <state_interface name="position"/>
-        </joint>
-    </ros2_control>
-    <!-- <ros2_control name="GazeboSystem" type="system">
-        <hardware>
-            <plugin>gazebo_ros2_control/GazeboSystem</plugin>
-        </hardware>
-        <joint name="rear_left_wheel_joint">
-            <command_interface name="velocity">
-                <param name="min">-1</param>
-                <param name="max">1</param>
-            </command_interface>
-            <state_interface name="velocity"/>
-        </joint>
-        <joint name="rear_right_wheel_joint">
-            <command_interface name="velocity">
-                <param name="min">-1</param>
-                <param name="max">1</param>
-            </command_interface>
-            <state_interface name="velocity"/>
-        </joint>
-        <joint name="front_left_steer_joint">
-            <command_interface name="position">
-                <param name="min">-0.5236</param>
-                <param name="max">0.5236</param>
-            </command_interface>
-            <state_interface name="position"/>
-        </joint>
-        <joint name="front_right_steer_joint">
-            <command_interface name="position">
-                <param name="min">-0.5236</param>
-                <param name="max">0.5236</param>
-            </command_interface>
-            <state_interface name="position"/>
-        </joint>
-    </ros2_control> -->
+    <xacro:unless value="$(arg sim_mode)">
+        <ros2_control name="RealRobot" type="system">
+            <hardware>
+                <plugin>doteacher/AckermannJetsonHardware</plugin>
+                <param name="rear_left_wheel">rear_left_wheel_joint</param>
+                <param name="rear_right_wheel">rear_right_wheel_joint</param>
+                <param name="front_left_wheel">front_left_steer_joint</param>
+                <param name="front_right_wheel">front_right_steer_joint</param>
+                <param name="loop_rate">20</param>
+            </hardware>
+            <joint name="rear_left_wheel_joint">
+                <command_interface name="velocity">
+                    <param name="min">-1</param>
+                    <param name="max">1</param>
+                </command_interface>
+                <state_interface name="velocity" />
+            </joint>
+            <joint name="rear_right_wheel_joint">
+                <command_interface name="velocity">
+                    <param name="min">-1</param>
+                    <param name="max">1</param>
+                </command_interface>
+                <state_interface name="velocity" />
+            </joint>
+            <joint name="front_left_steer_joint">
+                <command_interface name="position">
+                    <param name="min">-0.5236</param>
+                    <param name="max">0.5236</param>
+                </command_interface>
+                <state_interface name="position" />
+            </joint>
+            <joint name="front_right_steer_joint">
+                <command_interface name="position">
+                    <param name="min">-0.5236</param>
+                    <param name="max">0.5236</param>
+                </command_interface>
+                <state_interface name="position" />
+            </joint>
+        </ros2_control>
+    </xacro:unless>
+    <xacro:if value="$(arg sim_mode)">
+        <ros2_control name="GazeboSystem" type="system">
+            <hardware>
+                <plugin>gazebo_ros2_control/GazeboSystem</plugin>
+            </hardware>
+            <joint name="rear_left_wheel_joint">
+                <command_interface name="velocity">
+                    <param name="min">-1</param>
+                    <param name="max">1</param>
+                </command_interface>
+                <state_interface name="velocity" />
+            </joint>
+            <joint name="rear_right_wheel_joint">
+                <command_interface name="velocity">
+                    <param name="min">-1</param>
+                    <param name="max">1</param>
+                </command_interface>
+                <state_interface name="velocity" />
+            </joint>
+            <joint name="front_left_steer_joint">
+                <command_interface name="position">
+                    <param name="min">-0.5236</param>
+                    <param name="max">0.5236</param>
+                </command_interface>
+                <state_interface name="position" />
+            </joint>
+            <joint name="front_right_steer_joint">
+                <command_interface name="position">
+                    <param name="min">-0.5236</param>
+                    <param name="max">0.5236</param>
+                </command_interface>
+                <state_interface name="position" />
+            </joint>
+        </ros2_control>
+    </xacro:if>
     <gazebo>
         <plugin name="gazebo_ros2_control" filename="libgazebo_ros2_control.so">
             <parameters>$(find doteacher)/config/ros2_control/doteacher_controllers.yaml</parameters>
+            <parameters>$(find doteacher)/config/gazebo/gazebo_ros2_control_use_sim.yaml</parameters>
         </plugin>
     </gazebo>

File: ros/ros2_ws/src/doteacher/description/urdf/doteacher.urdf.xacro (robot description, xacro)
@@ -3,14 +3,17 @@
 <robot xmlns:xacro="http://www.ros.org/wiki/xacro" name="doteacher_robot">
   <xacro:arg name="prefix" default="" />
-  <xacro:arg name="use_ros2_control" default="true"/>
-  <xacro:arg name="sim_mode" default="false"/>
+  <xacro:arg name="use_ros2_control" default="true" />
+  <xacro:arg name="sim_mode" default="false" />
   <xacro:include filename="$(find doteacher)/urdf/doteacher_description.urdf.xacro" />
   <!-- Import Rviz colors -->
   <xacro:include filename="$(find doteacher)/urdf/doteacher.materials.xacro" />
   <xacro:ackermann prefix="$(arg prefix)" />
-  <!-- Import Gazebo control -->
-  <!-- <xacro:include filename="$(find doteacher)/gazebo_control/gazebo_ros_ackermann_drive.xacro"
-  /> -->
-  <!-- Import ros2 control -->
-  <xacro:include filename="$(find doteacher)/ros2_control/ros2_control_ackermann_drive.xacro" />
+  <xacro:if value="$(arg use_ros2_control)">
+    <!-- Import ros2 control -->
+    <xacro:include filename="$(find doteacher)/ros2_control/ros2_control_ackermann_drive.xacro" />
+  </xacro:if>
+  <xacro:unless value="$(arg use_ros2_control)">
+    <!-- Import Gazebo control -->
+    <xacro:include filename="$(find doteacher)/gazebo_control/gazebo_ros_ackermann_drive.xacro" />
+  </xacro:unless>
 </robot>

File: ros/ros2_ws/src/doteacher/description/urdf/doteacher_description.urdf.xacro (robot description, xacro)
@@ -13,5 +13,5 @@
     <xacro:property name="wheel_radius" value="0.0325" />
     <!-- <xacro:property name="wheeltrack" value="" -->
-    <xacro:property name="wheel_friction" value="0.8" />
+    <xacro:property name="wheel_friction" value="0.5" />
     <!-- Base Link -->
     <link name="${prefix}base_link" />
@@ -29,5 +29,5 @@
         <origin xyz="0 0 0" rpy="0 0 0" />
         <geometry>
-          <box size="${base_length} ${base_width} ${base_height}" />
+          <box size="${base_length} ${base_width-0.05} ${base_height}" />
         </geometry>
       </collision>
@@ -54,32 +54,17 @@
     </joint>
     <!-- steer -->
-    <!-- <link name="${prefix}steer_link"> -->
-      <!-- <visual>
-        <origin xyz="0 0 0.1" rpy="0 0 0" />
-        <geometry>
-          <cylinder length="0.05" radius="0.01" />
-        </geometry>
-        <material name="gold">
-          <color rgba="0.75 0.75 0.75 1" />
-        </material>
-      </visual>
-      <collision>
-        <origin xyz="0 0 0.1" rpy="0 0 0" />
-        <geometry>
-          <cylinder length="0.02" radius="0.01" />
-        </geometry>
-      </collision> -->
-      <!-- <inertial>
+    <!-- <link name="${prefix}steer_link">
+      <inertial>
         <mass value="0.001" />
         <inertia ixx="0.0" ixy="0.0" ixz="0.0" iyy="0.0" iyz="0.0" izz="0.0" />
       </inertial>
     </link>
-    <joint name="${prefix}steer_joint" type="prismatic">
+    <joint name="${prefix}steer_joint" type="revolute">
       <parent link="${prefix}chassis_link" />
       <child link="${prefix}steer_link" />
       <origin xyz="${wheelbase/2} 0 -${base_height/2}" rpy="0 0 0" />
-      <axis xyz="0 1 0" />
-      <limit lower="-0.005" upper="0.005" effort="5" velocity="0.0" />
-    </joint>-->
+      <axis xyz="1 0 0" />
+      <limit lower="-0.5236" upper="0.5236" effort="5" velocity="0.0" />
+    </joint> -->
     <link name="${prefix}front_left_hinge_link">
       <!-- <visual>
@@ -100,5 +85,8 @@
       <inertial>
         <mass value="0.001" />
-        <inertia ixx="0.0" ixy="0.0" ixz="0.0" iyy="0.0" iyz="0.0" izz="0.0" />
+        <inertia ixx="0.0001" ixy="0.000" ixz="0.000"
+          iyy="0.0001" iyz="0.000"
+          izz="0.0001"
+        />
       </inertial>
     </link>
@@ -109,5 +97,5 @@
       <axis xyz="0 0 1" />
       <limit lower="-0.5236" upper="0.5236" effort="5" velocity="0.0" />
-      <dynamics damping="0.0" friction="0.0" />
+      <dynamics damping="0.1" friction="0.0" />
     </joint>
     <link name="${prefix}front_right_hinge_link">
@@ -129,5 +117,6 @@
       <inertial>
         <mass value="0.001" />
-        <inertia ixx="0.0" ixy="0.0" ixz="0.0" iyy="0.0" iyz="0.0" izz="0.0" />
+        <inertia ixx="0.0001" ixy="0.000" ixz="0.000"
+          iyy="0.0001" iyz="0.000" izz="0.0001" />
       </inertial>
     </link>
@@ -138,5 +127,5 @@
       <axis xyz="0 0 1" />
       <limit lower="-0.5236" upper="0.5236" effort="5" velocity="0.0" />
-      <dynamics damping="0.0" friction="0.0" />
+      <dynamics damping="0.1" friction="0.0" />
     </joint>
     <!-- rear right wheel -->
@@ -170,5 +159,5 @@
       <axis xyz="0 0 -1" />
       <limit effort="10" velocity="10" />
-      <!-- <dynamics damping="0.2" /> -->
+      <dynamics damping="0.1" friction="0.0" />
     </joint>
     <!-- rear left wheel -->
@@ -202,5 +191,5 @@
       <axis xyz="0 0 1" />
       <limit effort="10" velocity="10" />
-      <!-- <dynamics damping="0.2" /> -->
+      <dynamics damping="0.1" friction="0.0" />
     </joint>
     <!-- front wheels -->
@@ -283,7 +272,10 @@
         </geometry>
       </collision>
-      <!-- <xacro:inertial_cylinder mass="0.1" radius="0.05" length="0.04">
-          <origin xyz="0 0 0" rpy="0 0 0" />
-      </xacro:inertial_cylinder> -->
+      <inertial>
+        <origin xyz="0 0 0" rpy="0 0 0" />
+        <mass value="0.05" />
+        <inertia ixx="0.0001" ixy="0.000" ixz="0.000"
+          iyy="0.0001" iyz="0.000" izz="0.0001" />
+      </inertial>
     </link>
     <!-- camera -->
@@ -300,12 +292,15 @@
         <material name="red" />
       </visual>
-      <!-- <collision>
-          <geometry>
-              <box size="0.010 0.03 0.03" />
-          </geometry>
-      </collision>
-      <xacro:inertial_box mass="0.1" size="0.010 0.03 0.03">
-          <origin xyz="0 0 0" rpy="0 0 0" />
-      </xacro:inertial_box> -->
+      <collision>
+        <geometry>
+          <box size="0.010 0.03 0.03" />
+        </geometry>
+      </collision>
+      <inertial>
+        <origin xyz="0 0 0" rpy="0 0 0" />
+        <mass value="0.01" />
+        <inertia ixx="0.0001" ixy="0.000" ixz="0.000"
+          iyy="0.0001" iyz="0.000" izz="0.0001" />
+      </inertial>
     </link>
     <joint name="${prefix}camera_optical_joint" type="fixed">
@@ -315,25 +310,46 @@
     </joint>
     <link name="${prefix}camera_link_optical">
+      <inertial>
+        <origin xyz="0 0 0" rpy="0 0 0" />
+        <mass value="0.000001" />
+        <inertia ixx="0.0001" ixy="0.000" ixz="0.000"
+          iyy="0.0001" iyz="0.000" izz="0.0001" />
+      </inertial>
     </link>
     <gazebo reference="base_link">
-      <dampingFactor>0.00007</dampingFactor>
     </gazebo>
     <gazebo reference="${prefix}chassis_link">
+      <damping>
+        <linear>0.2</linear>
+        <angular>0.05</angular>
+      </damping>
       <material>Gazebo/Orange</material>
     </gazebo>
     <gazebo reference="${prefix}rear_right_wheel">
-      <mu1>${wheel_friction}</mu1>
+      <mu1>0.5</mu1>
+      <mu2>0.5</mu2>
+      <kp>1000000.0</kp>
+      <kd>1.0</kd>
       <material>Gazebo/Black</material>
     </gazebo>
     <gazebo reference="${prefix}rear_left_wheel">
-      <mu1>${wheel_friction}</mu1>
+      <mu1>0.5</mu1>
+      <mu2>0.5</mu2>
+      <kp>1000000.0</kp>
+      <kd>1.0</kd>
       <material>Gazebo/Black</material>
     </gazebo>
     <gazebo reference="${prefix}front_right_wheel">
-      <mu1>${wheel_friction}</mu1>
+      <mu1>0.5</mu1>
+      <mu2>0.5</mu2>
+      <kp>1000000.0</kp>
+      <kd>1.0</kd>
       <material>Gazebo/Black</material>
     </gazebo>
     <gazebo reference="${prefix}front_left_wheel">
-      <mu1>${wheel_friction}</mu1>
+      <mu1>0.5</mu1>
+      <mu2>0.5</mu2>
+      <kp>1000000.0</kp>
+      <kd>1.0</kd>
       <material>Gazebo/Black</material>
     </gazebo>
