Commit message: Chore: urdf, params 변경

File: ros/ros2_ws/src/doteacher/description/ros2_control/doteacher.ros2_control.xacro (robot description, xacro)
@@ -7,4 +7,21 @@
         <param name="example_param_hw_start_duration_sec">0</param>
         <param name="example_param_hw_stop_duration_sec">3.0</param>
+        <param name="adj_steer">3</param>
+        <param name="adj_throttle_8_0">8.0</param>
+        <param name="adj_throttle_5_0">6.0</param>
+        <param name="adj_throttle_3_0">5.0</param>
+        <param name="adj_throttle_2_0">4.0</param>
+        <param name="adj_throttle_1_2">3.5</param>
+        <param name="adj_throttle_1_0">3.0</param>
+        <param name="adj_throttle_0_9">2.8</param>
+        <param name="adj_throttle_0_8">2.4</param>
+        <param name="adj_throttle_0_7">2.2</param>
+        <param name="adj_throttle_0_6">2.0</param>
+        <param name="adj_throttle_0_5">1.8</param>
+        <param name="adj_throttle_0_4">1.6</param>
+        <param name="adj_throttle_0_3">1.4</param>
+        <param name="adj_throttle_0_2">1.2</param>
+        <param name="adj_throttle_0_1">0.8</param>
+        <param name="adj_throttle_0_0">0.6</param>
       </hardware>
       <joint name="${prefix}virtual_front_wheel_joint">

File: ros/ros2_ws/src/doteacher/description/urdf/doteacher_description.urdf.xacro (robot description, xacro)
@@ -7,5 +7,5 @@
     <xacro:property name="base_width" value="0.125" />
     <xacro:property name="base_length" value="0.29" />
-    <xacro:property name="base_height" value="0.21" />
+    <xacro:property name="base_height" value="0.14" />
     <xacro:property name="wheelbase" value="0.135" />
     <xacro:property name="wheel_mass" value="0.05" /> <!-- arbitrary value for wheel mass -->
@@ -21,5 +21,5 @@
       <parent link="${prefix}base_link" />
       <child link="${prefix}base_footprint" />
-      <origin xyz="0 0 0" rpy="0 0 0" />
+      <origin xyz="0 0 -${wheel_radius}" rpy="0 0 0" />
       <axis xyz="0 0 1" />
     </joint>
@@ -27,5 +27,5 @@
     <link name="${prefix}chassis_link">
       <collision>
-        <origin xyz="0 0 0" rpy="0 0 0" />
+        <origin xyz="${base_length/2-0.01} 0 ${base_height/2}" rpy="0 0 0" />
         <geometry>
           <box size="${base_length} ${base_width} ${base_height}" />
@@ -33,5 +33,5 @@
       </collision>
       <visual>
-        <origin xyz="0 0 0" rpy="0 0 0" />
+        <origin xyz="${base_length/2-0.01} 0 ${base_height/2}" rpy="0 0 0" />
         <geometry>
           <box size="${base_length} ${base_width} ${base_height}" />
@@ -51,5 +51,5 @@
       <parent link="${prefix}base_link" />
       <child link="${prefix}chassis_link" />
-      <origin xyz="0 0 ${base_height/2 + wheel_radius}" rpy="0 0 0" />
+      <origin xyz="-0.090 0 0" rpy="0 0 0" />
       <axis xyz="0 0 1" />
       <dynamics damping="0.2" />
@@ -67,7 +67,7 @@
     </link>
     <joint name="${prefix}virtual_rear_wheel_joint" type="continuous">
-      <parent link="${prefix}chassis_link" />
+      <parent link="${prefix}base_link" />
       <child link="${prefix}virtual_rear_wheel" />
-      <origin xyz="-${wheelbase/2} 0 -${base_height/2}" rpy="0 0 ${PI/2}" />
+      <origin xyz="-${wheelbase/2} 0 0" rpy="0 0 ${PI/2}" />
       <axis xyz="1 0 0" />
       <limit effort="100.0" velocity="100.0" />
@@ -99,7 +99,7 @@
     </link>
     <joint name="${prefix}rear_right_wheel_joint" type="continuous">
-      <parent link="${prefix}chassis_link" />
+      <parent link="${prefix}base_link" />
       <child link="${prefix}rear_right_wheel" />
-      <origin xyz="-${wheelbase/2} ${base_width/2} -${base_height/2}" rpy="0 0 ${PI/2}" />
+      <origin xyz="-${wheelbase/2} ${base_width/2} 0" rpy="0 0 ${PI/2}" />
       <axis xyz="1 0 0" />
       <limit effort="100.0" velocity="100.0" />
@@ -132,7 +132,7 @@
     </link>
     <joint name="${prefix}rear_left_wheel_joint" type="continuous">
-      <parent link="${prefix}chassis_link" />
+      <parent link="${prefix}base_link" />
       <child link="${prefix}rear_left_wheel" />
-      <origin xyz="-${wheelbase/2} -${base_width/2} -${base_height/2}" rpy="0 0 ${PI/2}" />
+      <origin xyz="-${wheelbase/2} -${base_width/2} 0" rpy="0 0 ${PI/2}" />
       <axis xyz="1 0 0" />
       <limit effort="100.0" velocity="100.0" />
@@ -151,7 +151,7 @@
     </link>
     <joint name="${prefix}virtual_front_wheel_joint" type="revolute">
-      <parent link="${prefix}chassis_link" />
+      <parent link="${prefix}base_link" />
       <child link="${prefix}virtual_front_wheel" />
-      <origin xyz="${wheelbase/2} 0 -${base_height/2}" rpy="0 0 ${PI/2}" />
+      <origin xyz="${wheelbase/2} 0 0" rpy="0 0 ${PI/2}" />
       <axis xyz="0 0 1" />
       <limit lower="-0.4" upper="0.4" effort="100.0" velocity="0.0" />
@@ -161,66 +161,66 @@
     <link name="${prefix}front_right_wheel">
       <collision>
-        <origin xyz="0 0 0" rpy="${PI/2} 0 ${PI/2}"/>
-        <geometry>
-          <cylinder length="${wheel_len}" radius="${wheel_radius}"/>
-        </geometry>
-      </collision>
-      <visual>
-        <origin xyz="0 0 0" rpy="${PI/2} 0 ${PI/2}"/>
-        <geometry>
-          <cylinder length="${wheel_len}" radius="${wheel_radius}"/>
-        </geometry>
-        <material name="black"/>
-      </visual>
-      <inertial>
-        <origin xyz="0 0 0" rpy="${PI/2} 0 ${PI/2}"/>
-        <mass value="${wheel_mass}"/>
+        <origin xyz="0 0 0" rpy="${PI/2} 0 ${PI/2}" />
+        <geometry>
+          <cylinder length="${wheel_len}" radius="${wheel_radius}" />
+        </geometry>
+      </collision>
+      <visual>
+        <origin xyz="0 0 0" rpy="${PI/2} 0 ${PI/2}" />
+        <geometry>
+          <cylinder length="${wheel_len}" radius="${wheel_radius}" />
+        </geometry>
+        <material name="black" />
+      </visual>
+      <inertial>
+        <origin xyz="0 0 0" rpy="${PI/2} 0 ${PI/2}" />
+        <mass value="${wheel_mass}" />
         <inertia
           ixx="0.000270" ixy="0.0" ixz="0.0"
           iyy="0.000270" iyz="0.0"
-          izz="0.000426"/>
+          izz="0.000426" />
       </inertial>
     </link>
     <joint name="${prefix}front_right_wheel_joint" type="revolute">
-      <parent link="${prefix}chassis_link" />
+      <parent link="${prefix}base_link" />
       <child link="${prefix}front_right_wheel" />
-      <origin xyz="${wheelbase/2} ${base_width/2} -${base_height/2}" rpy="0 0 ${PI/2}"/>
-      <axis xyz="0 0 1"/>
-      <limit lower="-0.4" upper="0.4" effort="100.0" velocity="0.0"/>
-      <dynamics damping="0.2"/>
-      <mimic joint="${prefix}virtual_front_wheel_joint" multiplier="1.0" offset="0.0"/>
+      <origin xyz="${wheelbase/2} ${base_width/2} 0" rpy="0 0 ${PI/2}" />
+      <axis xyz="0 0 1" />
+      <limit lower="-0.4" upper="0.4" effort="100.0" velocity="0.0" />
+      <dynamics damping="0.2" />
+      <mimic joint="${prefix}virtual_front_wheel_joint" multiplier="1.0" offset="0.0" />
     </joint>
     <!-- front left wheel -->
     <link name="${prefix}front_left_wheel">
       <collision>
-        <origin xyz="0 0 0" rpy="${PI/2} 0 ${PI/2}"/>
-        <geometry>
-          <cylinder length="${wheel_len}" radius="${wheel_radius}"/>
-        </geometry>
-      </collision>
-      <visual>
-        <origin xyz="0 0 0" rpy="${PI/2} 0 ${PI/2}"/>
-        <geometry>
-          <cylinder length="${wheel_len}" radius="${wheel_radius}"/>
-        </geometry>
-        <material name="black"/>
-      </visual>
-      <inertial>
-        <origin xyz="0 0 0" rpy="${PI/2} 0 ${PI/2}"/>
-        <mass value="${wheel_mass}"/>
+        <origin xyz="0 0 0" rpy="${PI/2} 0 ${PI/2}" />
+        <geometry>
+          <cylinder length="${wheel_len}" radius="${wheel_radius}" />
+        </geometry>
+      </collision>
+      <visual>
+        <origin xyz="0 0 0" rpy="${PI/2} 0 ${PI/2}" />
+        <geometry>
+          <cylinder length="${wheel_len}" radius="${wheel_radius}" />
+        </geometry>
+        <material name="black" />
+      </visual>
+      <inertial>
+        <origin xyz="0 0 0" rpy="${PI/2} 0 ${PI/2}" />
+        <mass value="${wheel_mass}" />
         <inertia
           ixx="0.000270" ixy="0.0" ixz="0.0"
           iyy="0.000270" iyz="0.0"
-          izz="0.000426"/>
+          izz="0.000426" />
       </inertial>
     </link>
     <joint name="${prefix}front_left_wheel_joint" type="revolute">
-      <parent link="${prefix}chassis_link" />
+      <parent link="${prefix}base_link" />
       <child link="${prefix}front_left_wheel" />
-      <origin xyz="${wheelbase/2} -${base_width/2} -${base_height/2}" rpy="0 0 ${PI/2}"/>
-      <axis xyz="0 0 1"/>
-      <limit lower="-0.4" upper="0.4" effort="100.0" velocity="0.0"/>
-      <dynamics damping="0.2"/>
-      <mimic joint="${prefix}virtual_front_wheel_joint" multiplier="1.0" offset="0.0"/>
+      <origin xyz="${wheelbase/2} -${base_width/2} 0" rpy="0 0 ${PI/2}" />
+      <axis xyz="0 0 1" />
+      <limit lower="-0.4" upper="0.4" effort="100.0" velocity="0.0" />
+      <dynamics damping="0.2" />
+      <mimic joint="${prefix}virtual_front_wheel_joint" multiplier="1.0" offset="0.0" />
     </joint>
     <!-- lidar -->
@@ -228,5 +228,5 @@
       <parent link="${prefix}chassis_link" />
       <child link="${prefix}laser_frame" />
-      <origin xyz="0.05 0 ${base_height/2+0.005}" rpy="0 0 0" />
+      <origin xyz="0.180 0 0.195" rpy="0 0 0" />
     </joint>
     <link name="${prefix}laser_frame">
@@ -253,5 +253,5 @@
       <parent link="${prefix}chassis_link" />
       <child link="${prefix}camera_link" />
-      <origin xyz="${base_length/2} 0 0" rpy="0 0 0" />
+      <origin xyz="0.25 0 0.085" rpy="0 0 0" />
     </joint>
     <link name="${prefix}camera_link">
