Commit message: Chore: gazebo ackermann drive plugin 구현

File: ros/ros2_ws/src/doteacher/description/urdf/doteacher.urdf.xacro (robot description, xacro)
@@ -2,20 +2,10 @@
 <!-- 4 Wheel Robot with front steering and rear drive -->
 <robot xmlns:xacro="http://www.ros.org/wiki/xacro" name="doteacher_robot">
-  <xacro:arg name="use_ros2_control" default="true" />
-  <xacro:arg name="sim_mode" default="true" />
   <xacro:arg name="prefix" default="" />
   <xacro:include filename="$(find doteacher)/urdf/doteacher_description.urdf.xacro" />
   <!-- Import Rviz colors -->
   <xacro:include filename="$(find doteacher)/urdf/doteacher.materials.xacro" />
-  <xacro:if value="$(arg use_ros2_control)">
-    <!-- Import carlikebot ros2_control description -->
-    <xacro:include filename="$(find doteacher)/ros2_control/carlikebot.ros2_control.xacro" />
-    <xacro:carlikebot_ros2_control name="CarlikeBot" prefix="$(arg prefix)" />
-  </xacro:if>
-  <xacro:unless value="$(arg use_ros2_control)">
-    <!-- Import carlikebot gazebo description -->
-    <xacro:include
-      filename="$(find doteacher)/gazebo_control/carlikebot.gazebo_control.xacro" />
-  </xacro:unless>
-  <xacro:carlikebot prefix="$(arg prefix)" />
+  <xacro:ackermann prefix="$(arg prefix)" />
+  <!-- Import Gazebo control -->
+   <xacro:include filename="$(find doteacher)/gazebo_control/gazebo_ros_ackermann_drive.xacro" />
 </robot>

File: ros/ros2_ws/src/doteacher/description/urdf/doteacher_description.urdf.xacro (robot description, xacro)
@@ -1,8 +1,8 @@
 <?xml version="1.0"?>
 <robot xmlns:xacro="http://www.ros.org/wiki/xacro">
-  <xacro:macro name="carlikebot" params="prefix">
+  <xacro:macro name="ackermann" params="prefix">
     <!-- Constants for robot dimensions -->
     <xacro:property name="PI" value="3.1415926535897931" />
-    <xacro:property name="base_mass" value="4.0" /> <!-- arbitrary value for base mass -->
+    <xacro:property name="base_mass" value="2.0" /> <!-- arbitrary value for base mass -->
     <xacro:property name="base_width" value="0.125" />
     <xacro:property name="base_length" value="0.29" />
@@ -13,4 +13,5 @@
     <xacro:property name="wheel_radius" value="0.0325" />
     <!-- <xacro:property name="wheeltrack" value="" -->
+    <xacro:property name="wheel_friction" value="0.8" />
     <!-- Base Link -->
     <link name="${prefix}base_link" />
@@ -41,8 +42,7 @@
         <origin xyz="0 0 0" rpy="0 0 0" />
         <mass value="${base_mass}" />
-        <inertia
-          ixx="0.000270" ixy="0.0" ixz="0.0"
-          iyy="0.000270" iyz="0.0"
-          izz="0.000426" />
+        <inertia ixx="0.021367" ixy="0.0" ixz="0.0"
+          iyy="0.016621" iyz="0.0"
+          izz="0.009954" />
       </inertial>
     </link>
@@ -52,31 +52,91 @@
       <origin xyz="0 0 ${base_height/2 + wheel_radius}" rpy="0 0 0" />
       <axis xyz="0 0 1" />
-      <dynamics damping="0.2" />
-    </joint>
-    <gazebo reference="${prefix}chassis_link">
-      <material>Gazebo/Orange</material>
-    </gazebo>
-    <!-- rear wheels -->
-    <!-- virtual rear wheel -->
-    <link name="${prefix}virtual_rear_wheel">
-      <visual>
-        <origin xyz="0 0 0" rpy="${PI/2} 0 ${PI/2}" />
-        <geometry>
-          <cylinder length="0.01" radius="${wheel_radius}" />
-        </geometry>
-        <material name="invisible" />
-      </visual>
-      <inertial>
-        <mass value="2e-06"/>
-        <inertia ixx="1.1e-09" ixy="0" ixz="0" iyy="1.1e-09" iyz="0" izz="1.1e-09"/>
-      </inertial>
-    </link>
-    <joint name="${prefix}virtual_rear_wheel_joint" type="continuous">
-      <parent link="${prefix}chassis_link" />
-      <child link="${prefix}virtual_rear_wheel" />
-      <origin xyz="-${wheelbase/2} 0 -${base_height/2}" rpy="0 0 ${PI/2}" />
-      <axis xyz="1 0 0" />
-      <limit effort="100.0" velocity="100.0" />
-      <dynamics damping="0.2" />
+    </joint>
+    <!-- steer -->
+    <!-- <link name="${prefix}steer_link"> -->
+      <!-- <visual>
+        <origin xyz="0 0 0.1" rpy="0 0 0" />
+        <geometry>
+          <cylinder length="0.05" radius="0.01" />
+        </geometry>
+        <material name="gold">
+          <color rgba="0.75 0.75 0.75 1" />
+        </material>
+      </visual>
+      <collision>
+        <origin xyz="0 0 0.1" rpy="0 0 0" />
+        <geometry>
+          <cylinder length="0.02" radius="0.01" />
+        </geometry>
+      </collision> -->
+      <!-- <inertial>
+        <mass value="0.001" />
+        <inertia ixx="0.0" ixy="0.0" ixz="0.0" iyy="0.0" iyz="0.0" izz="0.0" />
+      </inertial>
+    </link>
+    <joint name="${prefix}steer_joint" type="prismatic">
+      <parent link="${prefix}chassis_link" />
+      <child link="${prefix}steer_link" />
+      <origin xyz="${wheelbase/2} 0 -${base_height/2}" rpy="0 0 0" />
+      <axis xyz="0 1 0" />
+      <limit lower="-0.005" upper="0.005" effort="5" velocity="0.0" />
+    </joint>-->
+    <link name="${prefix}front_left_hinge_link">
+      <!-- <visual>
+        <origin xyz="0 0 0.1" rpy="0 0 0" />
+        <geometry>
+          <cylinder length="0.05" radius="0.01" />
+        </geometry>
+        <material name="silver">
+          <color rgba="0.75 0.75 0.75 1" />
+        </material>
+      </visual>
+      <collision>
+        <origin xyz="0 0 0.1" rpy="0 0 0" />
+        <geometry>
+          <cylinder length="0.05" radius="0.01" />
+        </geometry>
+      </collision> -->
+      <inertial>
+        <mass value="0.001" />
+        <inertia ixx="0.0" ixy="0.0" ixz="0.0" iyy="0.0" iyz="0.0" izz="0.0" />
+      </inertial>
+    </link>
+    <joint name="${prefix}front_left_steer_joint" type="revolute">
+      <parent link="${prefix}chassis_link" />
+      <child link="${prefix}front_left_hinge_link" />
+      <origin xyz="${wheelbase/2} ${base_width/2} -${base_height/2}" rpy="0 0 0" />
+      <axis xyz="0 0 1" />
+      <limit lower="-0.5236" upper="0.5236" effort="5" velocity="0.0" />
+      <dynamics damping="0.0" friction="0.0" />
+    </joint>
+    <link name="${prefix}front_right_hinge_link">
+      <!-- <visual>
+        <origin xyz="0 0 0.1" rpy="0 0 0" />
+        <geometry>
+          <cylinder length="0.05" radius="0.01" />
+        </geometry>
+        <material name="silver">
+          <color rgba="0.75 0.75 0.75 1" />
+        </material>
+      </visual>
+      <collision>
+        <origin xyz="0 0 0.1" rpy="0 0 0" />
+        <geometry>
+          <cylinder length="0.05" radius="0.01" />
+        </geometry>
+      </collision> -->
+      <inertial>
+        <mass value="0.001" />
+        <inertia ixx="0.0" ixy="0.0" ixz="0.0" iyy="0.0" iyz="0.0" izz="0.0" />
+      </inertial>
+    </link>
+    <joint name="${prefix}front_right_steer_joint" type="revolute">
+      <parent link="${prefix}chassis_link" />
+      <child link="${prefix}front_right_hinge_link" />
+      <origin xyz="${wheelbase/2} -${base_width/2} -${base_height/2}" rpy="0 0 0" />
+      <axis xyz="0 0 1" />
+      <limit lower="-0.5236" upper="0.5236" effort="5" velocity="0.0" />
+      <dynamics damping="0.0" friction="0.0" />
     </joint>
     <!-- rear right wheel -->
@@ -104,7 +164,4 @@
       </inertial>
     </link>
-    <gazebo reference="${prefix}rear_right_wheel">
-      <material>Gazebo/Black</material>
-    </gazebo>
     <joint name="${prefix}rear_right_wheel_joint" type="continuous">
       <parent link="${prefix}chassis_link" />
@@ -112,7 +169,6 @@
       <origin xyz="-${wheelbase/2} ${base_width/2} -${base_height/2}" rpy="0 0 ${PI/2}" />
       <axis xyz="1 0 0" />
-      <limit effort="100.0" velocity="100.0" />
+      <limit effort="10" velocity="100.0" />
       <dynamics damping="0.2" />
-      <mimic joint="${prefix}virtual_rear_wheel_joint" multiplier="1.0" offset="0.0" />
     </joint>
     <!-- rear left wheel -->
@@ -140,7 +196,4 @@
       </inertial>
     </link>
-    <gazebo reference="${prefix}rear_left_wheel">
-      <material>Gazebo/Black</material>
-    </gazebo>
     <joint name="${prefix}rear_left_wheel_joint" type="continuous">
       <parent link="${prefix}chassis_link" />
@@ -148,41 +201,18 @@
       <origin xyz="-${wheelbase/2} -${base_width/2} -${base_height/2}" rpy="0 0 ${PI/2}" />
       <axis xyz="1 0 0" />
-      <limit effort="100.0" velocity="100.0" />
+      <limit effort="10" velocity="100.0" />
       <dynamics damping="0.2" />
-      <mimic joint="${prefix}virtual_rear_wheel_joint" multiplier="1.0" offset="0.0" />
     </joint>
     <!-- front wheels -->
-    <!-- virtual front wheel -->
-    <link name="${prefix}virtual_front_wheel">
-      <visual>
-        <origin xyz="0 0 0" rpy="${PI/2} 0 ${PI/2}" />
-        <geometry>
-          <cylinder length="0.01" radius="${wheel_radius}" />
-        </geometry>
-        <material name="invisible" />
-      </visual>
-      <inertial>
-        <mass value="2e-06"/>
-        <inertia ixx="1.1e-09" ixy="0" ixz="0" iyy="1.1e-09" iyz="0" izz="1.1e-09"/>
-      </inertial>
-    </link>
-    <joint name="${prefix}virtual_front_wheel_joint" type="revolute">
-      <parent link="${prefix}chassis_link" />
-      <child link="${prefix}virtual_front_wheel" />
-      <origin xyz="${wheelbase/2} 0 -${base_height/2}" rpy="0 0 ${PI/2}" />
-      <axis xyz="0 0 1" />
-      <limit lower="-0.4" upper="0.4" effort="100.0" velocity="0.0" />
-      <dynamics damping="0.2" />
-    </joint>
     <!-- front right wheel -->
     <link name="${prefix}front_right_wheel">
       <collision>
-        <origin xyz="0 0 0" rpy="${PI/2} 0 ${PI/2}" />
-        <geometry>
-          <cylinder length="${wheel_len}" radius="${wheel_radius}" />
-        </geometry>
-      </collision>
-      <visual>
-        <origin xyz="0 0 0" rpy="${PI/2} 0 ${PI/2}" />
+        <origin xyz="0 0 0" rpy="0 0 0" />
+        <geometry>
+          <cylinder length="${wheel_len}" radius="${wheel_radius}" />
+        </geometry>
+      </collision>
+      <visual>
+        <origin xyz="0 0 0" rpy="0 0 0" />
         <geometry>
           <cylinder length="${wheel_len}" radius="${wheel_radius}" />
@@ -191,5 +221,5 @@
       </visual>
       <inertial>
-        <origin xyz="0 0 0" rpy="${PI/2} 0 ${PI/2}" />
+        <origin xyz="0 0 0" rpy="0 0 0" />
         <mass value="${wheel_mass}" />
         <inertia
@@ -199,26 +229,20 @@
       </inertial>
     </link>
-    <gazebo reference="${prefix}front_right_wheel">
-      <material>Gazebo/Black</material>
-    </gazebo>
-    <joint name="${prefix}front_right_wheel_joint" type="revolute">
-      <parent link="${prefix}chassis_link" />
+    <joint name="${prefix}front_right_wheel_joint" type="continuous">
+      <parent link="${prefix}front_right_hinge_link" />
       <child link="${prefix}front_right_wheel" />
-      <origin xyz="${wheelbase/2} ${base_width/2} -${base_height/2}" rpy="0 0 ${PI/2}" />
-      <axis xyz="0 0 1" />
-      <limit lower="-0.4" upper="0.4" effort="100.0" velocity="0.0" />
-      <dynamics damping="0.2" />
-      <mimic joint="${prefix}virtual_front_wheel_joint" multiplier="1.0" offset="0.0" />
+      <origin xyz="0 0 0" rpy="-${PI/2} 0 0" />
+      <axis xyz="0 0 1" />
     </joint>
     <!-- front left steering -->
     <link name="${prefix}front_left_wheel">
       <collision>
-        <origin xyz="0 0 0" rpy="${PI/2} 0 ${PI/2}" />
-        <geometry>
-          <cylinder length="${wheel_len}" radius="${wheel_radius}" />
-        </geometry>
-      </collision>
-      <visual>
-        <origin xyz="0 0 0" rpy="${PI/2} 0 ${PI/2}" />
+        <origin xyz="0 0 0" rpy="0 0 0" />
+        <geometry>
+          <cylinder length="${wheel_len}" radius="${wheel_radius}" />
+        </geometry>
+      </collision>
+      <visual>
+        <origin xyz="0 0 0" rpy="0 0 0" />
         <geometry>
           <cylinder length="${wheel_len}" radius="${wheel_radius}" />
@@ -227,5 +251,5 @@
       </visual>
       <inertial>
-        <origin xyz="0 0 0" rpy="${PI/2} 0 ${PI/2}" />
+        <origin xyz="0 0 0" rpy="0 0 0" />
         <mass value="${wheel_mass}" />
         <inertia
@@ -235,16 +259,11 @@
       </inertial>
     </link>
-    <gazebo reference="${prefix}front_left_wheel">
-      <material>Gazebo/Black</material>
-    </gazebo>
-    <joint name="${prefix}front_left_wheel_joint" type="revolute">
-      <parent link="${prefix}chassis_link" />
+    <joint name="${prefix}front_left_wheel_joint" type="continuous">
+      <parent link="${prefix}front_left_hinge_link" />
       <child link="${prefix}front_left_wheel" />
-      <origin xyz="${wheelbase/2} -${base_width/2} -${base_height/2}" rpy="0 0 ${PI/2}" />
-      <axis xyz="0 0 1" />
-      <limit lower="-0.4" upper="0.4" effort="100.0" velocity="0.0" />
-      <dynamics damping="0.2" />
-      <mimic joint="${prefix}virtual_front_wheel_joint" multiplier="1.0" offset="0.0" />
-    </joint>
+      <origin xyz="0 0 0" rpy="${PI/2} 0 0" />
+      <axis xyz="0 0 1" />
+    </joint>
+    <!-- lidar -->
     <joint name="${prefix}laser_joint" type="fixed">
       <parent link="${prefix}chassis_link" />
@@ -268,7 +287,57 @@
       </xacro:inertial_cylinder> -->
     </link>
+    <!-- camera -->
+    <joint name="${prefix}camera_joint" type="fixed">
+      <parent link="${prefix}chassis_link" />
+      <child link="${prefix}camera_link" />
+      <origin xyz="${base_length/2} 0 0" rpy="0 0 0" />
+    </joint>
+    <link name="${prefix}camera_link">
+      <visual>
+        <geometry>
+          <box size="0.010 0.03 0.03" />
+        </geometry>
+        <material name="red" />
+      </visual>
+      <!-- <collision>
+          <geometry>
+              <box size="0.010 0.03 0.03" />
+          </geometry>
+      </collision>
+      <xacro:inertial_box mass="0.1" size="0.010 0.03 0.03">
+          <origin xyz="0 0 0" rpy="0 0 0" />
+      </xacro:inertial_box> -->
+    </link>
+    <joint name="${prefix}camera_optical_joint" type="fixed">
+      <parent link="${prefix}camera_link" />
+      <child link="${prefix}camera_link_optical" />
+      <origin xyz="0 0 0" rpy="${-pi/2} 0 ${-pi/2}" />
+    </joint>
+    <link name="${prefix}camera_link_optical">
+    </link>
+    <gazebo reference="base_link">
+      <dampingFactor>0.00007</dampingFactor>
+    </gazebo>
+    <gazebo reference="${prefix}chassis_link">
+      <material>Gazebo/Orange</material>
+    </gazebo>
+    <gazebo reference="${prefix}rear_right_wheel">
+      <mu1>${wheel_friction}</mu1>
+      <material>Gazebo/Black</material>
+    </gazebo>
+    <gazebo reference="${prefix}rear_left_wheel">
+      <mu1>${wheel_friction}</mu1>
+      <material>Gazebo/Black</material>
+    </gazebo>
+    <gazebo reference="${prefix}front_right_wheel">
+      <mu1>${wheel_friction}</mu1>
+      <material>Gazebo/Black</material>
+    </gazebo>
+    <gazebo reference="${prefix}front_left_wheel">
+      <mu1>${wheel_friction}</mu1>
+      <material>Gazebo/Black</material>
+    </gazebo>
     <gazebo reference="${prefix}laser_frame">
       <sensor name="laser" type="ray">
-        <always_on>true</always_on>
         <pose>0 0 0 0 0 0</pose>
         <visualize>false</visualize>
@@ -304,32 +373,4 @@
       <material>Gazebo/Red</material>
     </gazebo>
-    <joint name="${prefix}camera_joint" type="fixed">
-      <parent link="${prefix}chassis_link" />
-      <child link="${prefix}camera_link" />
-      <origin xyz="${base_length/2} 0 0" rpy="0 0 0" />
-    </joint>
-    <link name="${prefix}camera_link">
-      <visual>
-        <geometry>
-          <box size="0.010 0.03 0.03" />
-        </geometry>
-        <material name="red" />
-      </visual>
-      <!-- <collision>
-          <geometry>
-              <box size="0.010 0.03 0.03" />
-          </geometry>
-      </collision>
-      <xacro:inertial_box mass="0.1" size="0.010 0.03 0.03">
-          <origin xyz="0 0 0" rpy="0 0 0" />
-      </xacro:inertial_box> -->
-    </link>
-    <joint name="${prefix}camera_optical_joint" type="fixed">
-      <parent link="${prefix}camera_link" />
-      <child link="${prefix}camera_link_optical" />
-      <origin xyz="0 0 0" rpy="${-pi/2} 0 ${-pi/2}" />
-    </joint>
-    <link name="${prefix}camera_link_optical">
-    </link>
     <gazebo reference="${prefix}camera_link">
       <sensor name="camera" type="camera">

Commit message: Chore: gazebo ackermann custom controller 구현

File: ros/ros2_ws/src/doteacher/description/urdf/doteacher.urdf.xacro (robot description, xacro)
@@ -8,4 +8,7 @@
   <xacro:ackermann prefix="$(arg prefix)" />
   <!-- Import Gazebo control -->
-   <xacro:include filename="$(find doteacher)/gazebo_control/gazebo_ros_ackermann_drive.xacro" />
+  <!-- <xacro:include filename="$(find doteacher)/gazebo_control/gazebo_ros_ackermann_drive.xacro"
+  /> -->
+  <!-- Import ros2 control -->
+  <xacro:include filename="$(find doteacher)/ros2_control/ros2_control_ackermann_drive.xacro" />
 </robot>

File: ros/ros2_ws/src/doteacher/description/urdf/doteacher_description.urdf.xacro (robot description, xacro)
@@ -4,10 +4,10 @@
     <!-- Constants for robot dimensions -->
     <xacro:property name="PI" value="3.1415926535897931" />
-    <xacro:property name="base_mass" value="2.0" /> <!-- arbitrary value for base mass -->
+    <xacro:property name="base_mass" value="1.5" /> <!-- arbitrary value for base mass -->
     <xacro:property name="base_width" value="0.125" />
     <xacro:property name="base_length" value="0.29" />
     <xacro:property name="base_height" value="0.21" />
     <xacro:property name="wheelbase" value="0.135" />
-    <xacro:property name="wheel_mass" value="0.34055" /> <!-- arbitrary value for wheel mass -->
+    <xacro:property name="wheel_mass" value="0.05" /> <!-- arbitrary value for wheel mass -->
     <xacro:property name="wheel_len" value="0.02" />
     <xacro:property name="wheel_radius" value="0.0325" />
@@ -143,11 +143,11 @@
     <link name="${prefix}rear_right_wheel">
       <collision>
-        <origin xyz="0 0 0" rpy="${PI/2} 0 ${PI/2}" />
-        <geometry>
-          <cylinder length="${wheel_len}" radius="${wheel_radius}" />
-        </geometry>
-      </collision>
-      <visual>
-        <origin xyz="0 0 0" rpy="${PI/2} 0 ${PI/2}" />
+        <origin xyz="0 0 0" rpy="0 0 0" />
+        <geometry>
+          <cylinder length="${wheel_len}" radius="${wheel_radius}" />
+        </geometry>
+      </collision>
+      <visual>
+        <origin xyz="0 0 0" rpy="0 0 0" />
         <geometry>
           <cylinder length="${wheel_len}" radius="${wheel_radius}" />
@@ -156,5 +156,5 @@
       </visual>
       <inertial>
-        <origin xyz="0 0 0" rpy="${PI/2} 0 ${PI/2}" />
+        <origin xyz="0 0 0" rpy="0 0 0" />
         <mass value="${wheel_mass}" />
         <inertia
@@ -167,19 +167,19 @@
       <parent link="${prefix}chassis_link" />
       <child link="${prefix}rear_right_wheel" />
-      <origin xyz="-${wheelbase/2} ${base_width/2} -${base_height/2}" rpy="0 0 ${PI/2}" />
-      <axis xyz="1 0 0" />
-      <limit effort="10" velocity="100.0" />
-      <dynamics damping="0.2" />
+      <origin xyz="-${wheelbase/2} -${base_width/2} -${base_height/2}" rpy="${PI/2} 0 0" />
+      <axis xyz="0 0 -1" />
+      <limit effort="10" velocity="10" />
+      <!-- <dynamics damping="0.2" /> -->
     </joint>
     <!-- rear left wheel -->
     <link name="${prefix}rear_left_wheel">
       <collision>
-        <origin xyz="0 0 0" rpy="${PI/2} 0 ${PI/2}" />
-        <geometry>
-          <cylinder length="${wheel_len}" radius="${wheel_radius}" />
-        </geometry>
-      </collision>
-      <visual>
-        <origin xyz="0 0 0" rpy="${PI/2} 0 ${PI/2}" />
+        <origin xyz="0 0 0" rpy="0 0 0" />
+        <geometry>
+          <cylinder length="${wheel_len}" radius="${wheel_radius}" />
+        </geometry>
+      </collision>
+      <visual>
+        <origin xyz="0 0 0" rpy="0 0 0" />
         <geometry>
           <cylinder length="${wheel_len}" radius="${wheel_radius}" />
@@ -188,5 +188,5 @@
       </visual>
       <inertial>
-        <origin xyz="0 0 0" rpy="${PI/2} 0 ${PI/2}" />
+        <origin xyz="0 0 0" rpy="0 0 0" />
         <mass value="${wheel_mass}" />
         <inertia
@@ -199,8 +199,8 @@
       <parent link="${prefix}chassis_link" />
       <child link="${prefix}rear_left_wheel" />
-      <origin xyz="-${wheelbase/2} -${base_width/2} -${base_height/2}" rpy="0 0 ${PI/2}" />
-      <axis xyz="1 0 0" />
-      <limit effort="10" velocity="100.0" />
-      <dynamics damping="0.2" />
+      <origin xyz="-${wheelbase/2} ${base_width/2} -${base_height/2}" rpy="-${PI/2} 0 0" />
+      <axis xyz="0 0 1" />
+      <limit effort="10" velocity="10" />
+      <!-- <dynamics damping="0.2" /> -->
     </joint>
     <!-- front wheels -->
@@ -233,5 +233,5 @@
       <child link="${prefix}front_right_wheel" />
       <origin xyz="0 0 0" rpy="-${PI/2} 0 0" />
-      <axis xyz="0 0 1" />
+      <axis xyz="0 0 -1" />
     </joint>
     <!-- front left steering -->
@@ -262,5 +262,5 @@
       <parent link="${prefix}front_left_hinge_link" />
       <child link="${prefix}front_left_wheel" />
-      <origin xyz="0 0 0" rpy="${PI/2} 0 0" />
+      <origin xyz="0 0 0.00" rpy="-${PI/2} 0 0" />
       <axis xyz="0 0 1" />
     </joint>
@@ -312,5 +312,5 @@
       <parent link="${prefix}camera_link" />
       <child link="${prefix}camera_link_optical" />
-      <origin xyz="0 0 0" rpy="${-pi/2} 0 ${-pi/2}" />
+      <origin xyz="0 0 0" rpy="-${PI/2} 0 -${PI/2}" />
     </joint>
     <link name="${prefix}camera_link_optical">
