Commit message: Feat: ros2_control hardware interface 구현 완료

File: ros/ros2_ws/src/doteacher/description/urdf/doteacher.urdf.xacro (robot description, xacro)
@@ -3,17 +3,20 @@
 <robot xmlns:xacro="http://www.ros.org/wiki/xacro" name="doteacher_robot">
   <xacro:arg name="prefix" default="" />
-  <xacro:arg name="use_ros2_control" default="true" />
-  <xacro:arg name="sim_mode" default="false" />
+  <!-- <xacro:arg name="use_ros2_control" default="true" />
+  <xacro:arg name="sim_mode" default="false" /> -->
   <xacro:include filename="$(find doteacher)/urdf/doteacher_description.urdf.xacro" />
   <!-- Import Rviz colors -->
   <xacro:include filename="$(find doteacher)/urdf/doteacher.materials.xacro" />
-  <xacro:ackermann prefix="$(arg prefix)" />
+  doteacher
+  <!-- Import ros2 control -->
+  <xacro:include filename="$(find doteacher)/ros2_control/doteacher.ros2_control.xacro" />
+  <xacro:doteacher prefix="$(arg prefix)" />
+  <xacro:doteacher_ros2_control name="CarlikeBot" prefix="$(arg prefix)" />
+<!--
   <xacro:if value="$(arg use_ros2_control)">
-    <!-- Import ros2 control -->
-    <xacro:include filename="$(find doteacher)/ros2_control/ros2_control_carlike_drive.xacro" />
-  </xacro:if>
-  <xacro:unless value="$(arg use_ros2_control)">
+  </xacro:if> -->
+  <!-- <xacro:unless value="$(arg use_ros2_control)"> -->
     <!-- Import Gazebo control -->
-    <xacro:include filename="$(find doteacher)/gazebo_control/gazebo_ros_carlike_drive.xacro" />
-  </xacro:unless>
+    <!-- <xacro:include filename="$(find doteacher)/gazebo_control/gazebo_ros_carlike_drive.xacro" />
+  </xacro:unless> -->
 </robot>

File: ros/ros2_ws/src/doteacher/description/urdf/doteacher_description.urdf.xacro (robot description, xacro)
@@ -1,5 +1,5 @@
 <?xml version="1.0"?>
 <robot xmlns:xacro="http://www.ros.org/wiki/xacro">
-  <xacro:macro name="ackermann" params="prefix">
+  <xacro:macro name="doteacher" params="prefix">
     <!-- Constants for robot dimensions -->
     <xacro:property name="PI" value="3.1415926535897931" />
@@ -29,12 +29,12 @@
         <origin xyz="0 0 0" rpy="0 0 0" />
         <geometry>
-          <box size="${base_length} ${base_width-0.05} ${base_height}" />
-        </geometry>
-      </collision>
-      <visual>
-        <origin xyz="0 0 0" rpy="0 0 0" />
-        <geometry>
           <box size="${base_length} ${base_width} ${base_height}" />
         </geometry>
+      </collision>
+      <visual>
+        <origin xyz="0 0 0" rpy="0 0 0" />
+        <geometry>
+          <box size="${base_length} ${base_width} ${base_height}" />
+        </geometry>
         <material name="orange" />
       </visual>
@@ -42,5 +42,6 @@
         <origin xyz="0 0 0" rpy="0 0 0" />
         <mass value="${base_mass}" />
-        <inertia ixx="0.021367" ixy="0.0" ixz="0.0"
+        <inertia
+          ixx="0.021367" ixy="0.0" ixz="0.0"
           iyy="0.016621" iyz="0.0"
           izz="0.009954" />
@@ -52,85 +53,29 @@
       <origin xyz="0 0 ${base_height/2 + wheel_radius}" rpy="0 0 0" />
       <axis xyz="0 0 1" />
-    </joint>
-    <!-- steer -->
-    <!-- <link name="${prefix}steer_link">
-      <inertial>
-        <mass value="0.001" />
-        <inertia ixx="0.0" ixy="0.0" ixz="0.0" iyy="0.0" iyz="0.0" izz="0.0" />
-      </inertial>
-    </link>
-    <joint name="${prefix}steer_joint" type="revolute">
-      <parent link="${prefix}chassis_link" />
-      <child link="${prefix}steer_link" />
-      <origin xyz="${wheelbase/2} 0 -${base_height/2}" rpy="0 0 0" />
+      <dynamics damping="0.2" />
+    </joint>
+    <!-- rear wheels -->
+    <!-- virtual rear wheel -->
+    <link name="${prefix}virtual_rear_wheel">
+      <visual>
+        <origin xyz="0 0 0" rpy="${PI/2} 0 ${PI/2}" />
+        <geometry>
+          <cylinder length="0.01" radius="${wheel_radius}" />
+        </geometry>
+        <material name="invisible" />
+      </visual>
+    </link>
+    <joint name="${prefix}virtual_rear_wheel_joint" type="continuous">
+      <parent link="${prefix}chassis_link" />
+      <child link="${prefix}virtual_rear_wheel" />
+      <origin xyz="-${wheelbase/2} 0 -${base_height/2}" rpy="0 0 ${PI/2}" />
       <axis xyz="1 0 0" />
-      <limit lower="-0.5236" upper="0.5236" effort="5" velocity="0.0" />
-    </joint> -->
-    <link name="${prefix}front_left_hinge_link">
-      <!-- <visual>
-        <origin xyz="0 0 0.1" rpy="0 0 0" />
-        <geometry>
-          <cylinder length="0.05" radius="0.01" />
-        </geometry>
-        <material name="silver">
-          <color rgba="0.75 0.75 0.75 1" />
-        </material>
-      </visual>
-      <collision>
-        <origin xyz="0 0 0.1" rpy="0 0 0" />
-        <geometry>
-          <cylinder length="0.05" radius="0.01" />
-        </geometry>
-      </collision> -->
-      <inertial>
-        <mass value="0.001" />
-        <inertia ixx="0.0001" ixy="0.000" ixz="0.000"
-          iyy="0.0001" iyz="0.000"
-          izz="0.0001"
-        />
-      </inertial>
-    </link>
-    <joint name="${prefix}front_left_steer_joint" type="revolute">
-      <parent link="${prefix}chassis_link" />
-      <child link="${prefix}front_left_hinge_link" />
-      <origin xyz="${wheelbase/2} ${base_width/2} -${base_height/2}" rpy="0 0 0" />
-      <axis xyz="0 0 1" />
-      <limit lower="-0.5236" upper="0.5236" effort="5" velocity="0.0" />
-      <dynamics damping="0.1" friction="0.0" />
-    </joint>
-    <link name="${prefix}front_right_hinge_link">
-      <!-- <visual>
-        <origin xyz="0 0 0.1" rpy="0 0 0" />
-        <geometry>
-          <cylinder length="0.05" radius="0.01" />
-        </geometry>
-        <material name="silver">
-          <color rgba="0.75 0.75 0.75 1" />
-        </material>
-      </visual>
-      <collision>
-        <origin xyz="0 0 0.1" rpy="0 0 0" />
-        <geometry>
-          <cylinder length="0.05" radius="0.01" />
-        </geometry>
-      </collision> -->
-      <inertial>
-        <mass value="0.001" />
-        <inertia ixx="0.0001" ixy="0.000" ixz="0.000"
-          iyy="0.0001" iyz="0.000" izz="0.0001" />
-      </inertial>
-    </link>
-    <joint name="${prefix}front_right_steer_joint" type="revolute">
-      <parent link="${prefix}chassis_link" />
-      <child link="${prefix}front_right_hinge_link" />
-      <origin xyz="${wheelbase/2} -${base_width/2} -${base_height/2}" rpy="0 0 0" />
-      <axis xyz="0 0 1" />
-      <limit lower="-0.5236" upper="0.5236" effort="5" velocity="0.0" />
-      <dynamics damping="0.1" friction="0.0" />
+      <limit effort="100.0" velocity="100.0" />
+      <dynamics damping="0.2" />
     </joint>
     <!-- rear right wheel -->
     <link name="${prefix}rear_right_wheel">
       <collision>
-        <origin xyz="0 0 0" rpy="0 0 0" />
+        <origin xyz="0 0 0" rpy="${PI/2} 0 ${PI/2}" />
         <geometry>
           <cylinder length="${wheel_len}" radius="${wheel_radius}" />
@@ -138,5 +83,5 @@
       </collision>
       <visual>
-        <origin xyz="0 0 0" rpy="0 0 0" />
+        <origin xyz="0 0 0" rpy="${PI/2} 0 ${PI/2}" />
         <geometry>
           <cylinder length="${wheel_len}" radius="${wheel_radius}" />
@@ -145,5 +90,5 @@
       </visual>
       <inertial>
-        <origin xyz="0 0 0" rpy="0 0 0" />
+        <origin xyz="0 0 0" rpy="${PI/2} 0 ${PI/2}" />
         <mass value="${wheel_mass}" />
         <inertia
@@ -156,13 +101,14 @@
       <parent link="${prefix}chassis_link" />
       <child link="${prefix}rear_right_wheel" />
-      <origin xyz="-${wheelbase/2} -${base_width/2} -${base_height/2}" rpy="${PI/2} 0 0" />
-      <axis xyz="0 0 -1" />
-      <limit effort="10" velocity="10" />
-      <dynamics damping="0.1" friction="0.0" />
+      <origin xyz="-${wheelbase/2} ${base_width/2} -${base_height/2}" rpy="0 0 ${PI/2}" />
+      <axis xyz="1 0 0" />
+      <limit effort="100.0" velocity="100.0" />
+      <dynamics damping="0.2" />
+      <mimic joint="${prefix}virtual_rear_wheel_joint" multiplier="1.0" offset="0.0" />
     </joint>
     <!-- rear left wheel -->
     <link name="${prefix}rear_left_wheel">
       <collision>
-        <origin xyz="0 0 0" rpy="0 0 0" />
+        <origin xyz="0 0 0" rpy="${PI/2} 0 ${PI/2}" />
         <geometry>
           <cylinder length="${wheel_len}" radius="${wheel_radius}" />
@@ -170,5 +116,5 @@
       </collision>
       <visual>
-        <origin xyz="0 0 0" rpy="0 0 0" />
+        <origin xyz="0 0 0" rpy="${PI/2} 0 ${PI/2}" />
         <geometry>
           <cylinder length="${wheel_len}" radius="${wheel_radius}" />
@@ -177,5 +123,5 @@
       </visual>
       <inertial>
-        <origin xyz="0 0 0" rpy="0 0 0" />
+        <origin xyz="0 0 0" rpy="${PI/2} 0 ${PI/2}" />
         <mass value="${wheel_mass}" />
         <inertia
@@ -188,69 +134,93 @@
       <parent link="${prefix}chassis_link" />
       <child link="${prefix}rear_left_wheel" />
-      <origin xyz="-${wheelbase/2} ${base_width/2} -${base_height/2}" rpy="-${PI/2} 0 0" />
+      <origin xyz="-${wheelbase/2} -${base_width/2} -${base_height/2}" rpy="0 0 ${PI/2}" />
+      <axis xyz="1 0 0" />
+      <limit effort="100.0" velocity="100.0" />
+      <dynamics damping="0.2" />
+      <mimic joint="${prefix}virtual_rear_wheel_joint" multiplier="1.0" offset="0.0" />
+    </joint>
+    <!-- front wheels -->
+    <link name="${prefix}virtual_front_wheel">
+      <visual>
+        <origin xyz="0 0 0" rpy="${PI/2} 0 ${PI/2}" />
+        <geometry>
+          <cylinder length="0.01" radius="${wheel_radius}" />
+        </geometry>
+        <material name="invisible" />
+      </visual>
+    </link>
+    <joint name="${prefix}virtual_front_wheel_joint" type="revolute">
+      <parent link="${prefix}chassis_link" />
+      <child link="${prefix}virtual_front_wheel" />
+      <origin xyz="${wheelbase/2} 0 -${base_height/2}" rpy="0 0 ${PI/2}" />
       <axis xyz="0 0 1" />
-      <limit effort="10" velocity="10" />
-      <dynamics damping="0.1" friction="0.0" />
-    </joint>
-    <!-- front wheels -->
+      <limit lower="-0.4" upper="0.4" effort="100.0" velocity="0.0" />
+      <dynamics damping="0.2" />
+    </joint>
     <!-- front right wheel -->
     <link name="${prefix}front_right_wheel">
       <collision>
-        <origin xyz="0 0 0" rpy="0 0 0" />
-        <geometry>
-          <cylinder length="${wheel_len}" radius="${wheel_radius}" />
-        </geometry>
-      </collision>
-      <visual>
-        <origin xyz="0 0 0" rpy="0 0 0" />
-        <geometry>
-          <cylinder length="${wheel_len}" radius="${wheel_radius}" />
-        </geometry>
-        <material name="black" />
-      </visual>
-      <inertial>
-        <origin xyz="0 0 0" rpy="0 0 0" />
-        <mass value="${wheel_mass}" />
+        <origin xyz="0 0 0" rpy="${PI/2} 0 ${PI/2}"/>
+        <geometry>
+          <cylinder length="${wheel_len}" radius="${wheel_radius}"/>
+        </geometry>
+      </collision>
+      <visual>
+        <origin xyz="0 0 0" rpy="${PI/2} 0 ${PI/2}"/>
+        <geometry>
+          <cylinder length="${wheel_len}" radius="${wheel_radius}"/>
+        </geometry>
+        <material name="black"/>
+      </visual>
+      <inertial>
+        <origin xyz="0 0 0" rpy="${PI/2} 0 ${PI/2}"/>
+        <mass value="${wheel_mass}"/>
         <inertia
           ixx="0.000270" ixy="0.0" ixz="0.0"
           iyy="0.000270" iyz="0.0"
-          izz="0.000426" />
-      </inertial>
-    </link>
-    <joint name="${prefix}front_right_wheel_joint" type="continuous">
-      <parent link="${prefix}front_right_hinge_link" />
+          izz="0.000426"/>
+      </inertial>
+    </link>
+    <joint name="${prefix}front_right_wheel_joint" type="revolute">
+      <parent link="${prefix}chassis_link" />
       <child link="${prefix}front_right_wheel" />
-      <origin xyz="0 0 0" rpy="-${PI/2} 0 0" />
-      <axis xyz="0 0 -1" />
-    </joint>
-    <!-- front left steering -->
+      <origin xyz="${wheelbase/2} ${base_width/2} -${base_height/2}" rpy="0 0 ${PI/2}"/>
+      <axis xyz="0 0 1"/>
+      <limit lower="-0.4" upper="0.4" effort="100.0" velocity="0.0"/>
+      <dynamics damping="0.2"/>
+      <mimic joint="${prefix}virtual_front_wheel_joint" multiplier="1.0" offset="0.0"/>
+    </joint>
+    <!-- front left wheel -->
     <link name="${prefix}front_left_wheel">
       <collision>
-        <origin xyz="0 0 0" rpy="0 0 0" />
-        <geometry>
-          <cylinder length="${wheel_len}" radius="${wheel_radius}" />
-        </geometry>
-      </collision>
-      <visual>
-        <origin xyz="0 0 0" rpy="0 0 0" />
-        <geometry>
-          <cylinder length="${wheel_len}" radius="${wheel_radius}" />
-        </geometry>
-        <material name="black" />
-      </visual>
-      <inertial>
-        <origin xyz="0 0 0" rpy="0 0 0" />
-        <mass value="${wheel_mass}" />
+        <origin xyz="0 0 0" rpy="${PI/2} 0 ${PI/2}"/>
+        <geometry>
+          <cylinder length="${wheel_len}" radius="${wheel_radius}"/>
+        </geometry>
+      </collision>
+      <visual>
+        <origin xyz="0 0 0" rpy="${PI/2} 0 ${PI/2}"/>
+        <geometry>
+          <cylinder length="${wheel_len}" radius="${wheel_radius}"/>
+        </geometry>
+        <material name="black"/>
+      </visual>
+      <inertial>
+        <origin xyz="0 0 0" rpy="${PI/2} 0 ${PI/2}"/>
+        <mass value="${wheel_mass}"/>
         <inertia
           ixx="0.000270" ixy="0.0" ixz="0.0"
           iyy="0.000270" iyz="0.0"
-          izz="0.000426" />
-      </inertial>
-    </link>
-    <joint name="${prefix}front_left_wheel_joint" type="continuous">
-      <parent link="${prefix}front_left_hinge_link" />
+          izz="0.000426"/>
+      </inertial>
+    </link>
+    <joint name="${prefix}front_left_wheel_joint" type="revolute">
+      <parent link="${prefix}chassis_link" />
       <child link="${prefix}front_left_wheel" />
-      <origin xyz="0 0 0.00" rpy="-${PI/2} 0 0" />
-      <axis xyz="0 0 1" />
+      <origin xyz="${wheelbase/2} -${base_width/2} -${base_height/2}" rpy="0 0 ${PI/2}"/>
+      <axis xyz="0 0 1"/>
+      <limit lower="-0.4" upper="0.4" effort="100.0" velocity="0.0"/>
+      <dynamics damping="0.2"/>
+      <mimic joint="${prefix}virtual_front_wheel_joint" multiplier="1.0" offset="0.0"/>
     </joint>
     <!-- lidar -->
