Commit message: Feat: nav2 연동 완료

File: ros/ros2_ws/src/doteacher/description/urdf/doteacher_description.urdf.xacro (robot description, xacro)
@@ -228,5 +228,5 @@
       <parent link="${prefix}chassis_link" />
       <child link="${prefix}laser_frame" />
-      <origin xyz="0.05 0 ${base_height/2+0.005}" rpy="0 0 ${PI}" />
+      <origin xyz="0.05 0 ${base_height/2+0.005}" rpy="0 0 0" />
     </joint>
     <link name="${prefix}laser_frame">
